File: PowerCircuit_v1/PowerCircuit_v1.kicad_pcb (KiCad board)
At the start: 2 copper layers, 98 x 98 mm, 20 parts, among them U1 MPD7K020S

Commit message: Add files via upload
Parts:
- added G***: LOGO, Library:sken, F.Cu at (126.1, 85.4)
Other:
- board text added: "2024/02/14"
- board text added: "JLCJLCJLCJLC"
- board text added: "https://github.com/makizusi/-circuit"
- board text added: "makizusi_PowerCircuit_v1"
