File: sensor_v1/sensor_v1.kicad_pcb (KiCad board)
At the start: 2 copper layers, 98.1 x 98 mm, 43 parts, among them J1 LS, J10 stlink, J11 USB_A, J12 USB_B, J13 Conn_01x04, J14 Conn_01x04, J15 LS, J16 LS, J17 LS, J2 LS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

Commit message: Add files via upload
Other:
- board text added: "2024/02/14"
- board text added: "https://github.com/makizusi/-circuit"
- board text added: "makizusi_sensor_v1"
